File: HW/V2.1/cpu.sch (KiCad schematic (older format))
At the start: 78 parts, among them Q1 FDN360P, Q4 FDN360P, T2 Panasonic_EVQPUL_EVQPUC, U1 STM32F334, U2 MIC5501-3.0V, U3 BY25Q64ASSIG, U5 ESP8266EX, U6 BS801B, X1 TC2050-IDC, X3 TC2050-IDC

Commit message: fixed values
Parts:
- added C59: 18p 50V, Capacitor_SMD:C_0603_1608Metric, symbol EO:C-0402-18p-50V
- C11, C15: value 82n -> 47n
- C46: value 18p 50V -> DNP
Connections:
- net GND: now also C59.1
- net TOUCH7: now also C59.2
Changed lines of the file:
@@
 EESchema Schematic File Version 4
-LIBS:main-cache
 EELAYER 30 0
 EELAYER END
@@
 P 1950 7100
 F 0 "C15" H 2000 6837 60  0000 C CNN
-F 1 "82n" H 2000 6731 60  0000 C CNN
+F 1 "47n" H 2000 6731 60  0000 C CNN
 F 2 "Capacitor_SMD:C_0603_1608Metric" H 1940 6810 60  0001 C CNN
 F 3 "" H 1940 6810 60  0000 C CNN
@@
 P 1950 6700
 F 0 "C11" H 2000 6869 60  0000 C CNN
-F 1 "82n" H 2000 6763 60  0000 C CNN
+F 1 "47n" H 2000 6763 60  0000 C CNN
 F 2 "Capacitor_SMD:C_0603_1608Metric" H 1940 6410 60  0001 C CNN
 F 3 "" H 1940 6410 60  0000 C CNN
@@
 	1    0    0    -1
 $EndComp
-Text GLabel 7800 5150 0    50   Input ~ 0
+Text GLabel 7600 5150 0    50   Input ~ 0
 TOUCH7
 $Comp
@@
 P 8750 5350
 F 0 "C46" V 8853 5140 60  0000 R CNN
-F 1 "18p 50V" V 8747 5140 60  0000 R CNN
+F 1 "DNP" V 8747 5140 60  0000 R CNN
 F 2 "Capacitor_SMD:C_0603_1608Metric" H 8860 5440 60  0001 C CNN
 F 3 "" H 8860 5440 60  0000 C CNN
@@
 Wire Wire Line
 	5700 3150 6700 3150
+$Comp
+L EO:C-0402-18p-50V C59
+U 1 1 5E7D8249
+P 7600 5400
+F 0 "C59" V 7703 5190 60  0000 R CNN
+F 1 "18p 50V" V 7597 5190 60  0000 R CNN
+F 2 "Capacitor_SMD:C_0603_1608Metric" H 7710 5490 60  0001 C CNN
+F 3 "" H 7710 5490 60  0000 C CNN
+	1    7600 5400
+	0    -1   -1   0
+$EndComp
+$Comp
+L power:GND #GND0149
+U 1 1 5E7D824F
+P 7700 5500
+F 0 "#GND0149" H 7788 5493 20  0000 L CNN
+F 1 "GND" H 7788 5441 30  0000 L CNN
+F 2 "" H 7700 5500 70  0000 C CNN
+F 3 "" H 7700 5500 70  0000 C CNN
+	1    7700 5500
+	1    0    0    -1
+$EndComp
+Wire Wire Line
+	7800 5150 7700 5150
+Wire Wire Line
+	7700 5150 7700 5200
+Wire Wire Line
+	7700 5150 7600 5150
+Connection ~ 7700 5150
 $EndSCHEMATC
