File: HW/V2.1/main.kicad_pcb (KiCad board)
At the start: 2 copper layers, 100 x 100 mm, 181 parts, among them IC1 RT9466, IC2 MIC4416, IC3 MIC4416, J4 USB-C, Q1 FDN360P, Q2 NTMS4816NR2G, Q3 NTMS4816NR2G, Q4 FDN360P, T2 Panasonic_EVQPUL_EVQPUC, U1 STM32F334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

Commit message: fixed values
Parts:
- added C59: 18p 50V, Capacitor_SMD:C_0603_1608Metric, B.Cu at (116.8, 107.8)
- 254_1, 254_2: value Val** -> 254
- C11, C15: value 82n -> 47n
- C46: value 18p 50V -> DNP
- L2, L3: value 4.7u -> 4.7u 3.5A
- R29: value 698 -> 300
- R33: value 47k -> 220k
- R35, R38: value 5 -> 6.2
Routing:
- net GND: track 610.8 -> 612.6 mm, vias 167 -> 166
- net TOUCH7: track 19.5 -> 20.8 mm
